File: Battery Gauge Main Board.brd (EAGLE design)
At the start: 18.9 x 11.9 mm, 21 parts, among them J1 AVR_SPI_6, U3 TINY48

Commit message: Updated parts list
Parts:
- U3: value TINY48 -> ATtiny48-MMU
Changed lines of the file:
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@@
 <element name="LIPO-" library="SparkFun" package="1X01_SMD_SMALL" value="M01SMALL" x="17.65" y="8.6" rot="R270"/>
 <element name="R6" library="adafruit" package="R0603_S" value="10K" x="11.9" y="14.6"/>
-<element name="U3" library="avr-5" package="VQFN-28" value="TINY48" x="16.35" y="14.05" rot="R90"/>
+<element name="U3" library="avr-5" package="VQFN-28" value="ATtiny48-MMU" x="16.35" y="14.05" rot="R90"/>
 <element name="C3" library="adafruit" package="C0603K" value="0.1uF" x="16.35" y="17.65" rot="R180"/>
 <element name="C4" library="adafruit" package="C0603K" value="0.1uF" x="16.2" y="10.2"/>
