File: Battery Gauge Main Board.sch (EAGLE design)
At the start: 21 parts, among them J1 AVR_SPI_6, U3 TINY48

Commit message: Updated parts list
Parts:
- U3: value TINY48 -> ATtiny48-MMU
Changed lines of the file:
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@@
 <part name="GND2" library="SparkFun" deviceset="GND" device=""/>
 <part name="R6" library="adafruit" deviceset="R-US_" device="R0603_S" value="10K"/>
-<part name="U3" library="avr-5" deviceset="TINY48" device=""/>
+<part name="U3" library="avr-5" deviceset="TINY48" device="" value="ATtiny48-MMU"/>
 <part name="GND6" library="SparkFun" deviceset="GND" device=""/>
 <part name="C3" library="adafruit" deviceset="CAP" device="0603" value="0.1uF"/>
